Commit message: teleop update

File: rover_description/urdf/rover.urdf.xacro (robot description, xacro)
@@ -26,8 +26,7 @@
   <xacro:include filename="$(find rover_description)/urdf/wheel.urdf.xacro" />
   <xacro:include filename="$(find rover_description)/urdf/accessories/kinect_camera.urdf.xacro"/>
-  <xacro:include filename="$(find rover_description)/urdf/accessories/sick_lms1xx_mount.urdf.xacro"/>
   <xacro:include filename="$(find rover_description)/urdf/accessories/sensor_arch.urdf.xacro"/>
   <xacro:include filename="$(find rover_description)/urdf/accessories/camera.urdf.xacro"/>
-  <xacro:include filename="$(find ur_description)/urdf/ur5.urdf.xacro" />
+  <xacro:include filename="$(find ouster_description)/urdf/OS1-64.urdf.xacro"/>
   <property name="M_PI" value="3.14159"/>
   <!-- Base Size -->
@@ -95,4 +94,13 @@
     <gazebo reference="imu_link">
     </gazebo>
+    <!-- GPS link -->
+    <link name="navsat_link"/>
+    <joint name="navsat_joint" type="fixed">
+      <parent link="base_link" />
+      <child link="navsat_link" />
+      <origin xyz="0.19 0 0.149" rpy="0 -1.5708 3.1416" />
+    </joint>
+    <gazebo reference="navsat_link">
+    </gazebo>
     <!-- Wheel macros -->
     <xacro:rover_wheel wheel_prefix="front_left">
@@ -109,24 +117,4 @@
     </xacro:rover_wheel>
    <xacro:rover_decorate />
-    <xacro:if value="$(arg ur5_enabled)">
-      <xacro:property name="reflect" value="-1" />
-      <!-- Spawn arm -->
-      <xacro:ur5_robot prefix="ur5_arm_" joint_limited="true"/>
-      <!-- Join arm -->
-      <joint name="ur5_arm_base" type="fixed">
-        <parent link="top_plate_link" />
-        <child link="ur5_arm_base_link" />
-        <origin xyz="0.3058 0 0.0065" rpy="0.0 0.0 -1.57" />
-      </joint>
-    </xacro:if>
-    <xacro:if value="$(arg laser_enabled)">
-      <sick_lms1xx_mount prefix="base" topic="scan"/>
-      <joint name="laser_mount_joint" type="fixed">
-        <!-- <origin xyz="$(optenv HUSKY_LMS1XX_XYZ 0.2206 0.0 0.00635)" rpy="$(optenv HUSKY_LMS1XX_RPY 0.0 0.0 0.0)" /> -->
-	<origin xyz="0.2206 0.0 0.00635" rpy="0.0 0.0 0.0" />
-        <parent link="top_plate_link" />
-        <child link="base_laser_mount" />
-      </joint>
-    </xacro:if>
     <xacro:if value="$(arg kinect_enabled)">
       <xacro:sensor_arch prefix="" parent="top_plate_link">
@@ -162,4 +150,16 @@
     </xacro:camera_macro>
   </xacro:if>
+  <!--Mount a OS1-64-->
+  <xacro:if value="$(arg os1-64_enabled)">
+    <xacro:OS1-64
+      parent="base_link"
+      name="ouster"
+      topic="/points"
+      hz="10"
+      samples="220"
+    >
+    <origin xyz="0 0 0.02" rpy="0 0 0" />
+    </xacro:OS1-64>
+  </xacro:if>
   </xacro:macro>
 </robot>

File: rover_description/urdf/wheel.urdf.xacro (robot description, xacro)
@@ -61,5 +61,5 @@
 			</actuator>
 			<joint name="${wheel_prefix}_wheel">
-				<hardwareInterface>VelocityJointInterface</hardwareInterface>
+				<hardwareInterface>hardware_interface/VelocityJointInterface</hardwareInterface>
 			</joint>
 		</transmission>

File: rover_gazebo/urdf/rover.gazebo.xacro (robot description, xacro)
@@ -28,6 +28,6 @@
         <robotNamespace>/</robotNamespace>
         <updateRate>50.0</updateRate>
-        <bodyName>base_link</bodyName>
-        <topicName>imu/data</topicName>
+        <bodyName>imu_link</bodyName>
+        <topicName>imu/data_raw</topicName>
         <accelDrift>0.005 0.005 0.005</accelDrift>
         <accelGaussianNoise>0.005 0.005 0.005</accelGaussianNoise>
@@ -42,7 +42,7 @@
         <updateRate>40</updateRate>
         <robotNamespace>/</robotNamespace>
-        <bodyName>base_link</bodyName>
+        <bodyName>navsat_link</bodyName>
         <frameId>base_link</frameId>
-        <topicName>navsat/fix</topicName>
+        <topicName>navsat/fix_raw</topicName>
         <velocityTopicName>navsat/vel</velocityTopicName>
         <referenceLatitude>49.9</referenceLatitude>

File: rover_gazebo/urdf/rover_description.gazebo.xacro (robot description, xacro)
@@ -26,6 +26,7 @@
   <xacro:arg name="ur5_enabled" default="false" />
   <xacro:arg name="kinect_enabled" default="false" />
+  <xacro:arg name="os1-64_enabled" default="false" />
   <xacro:include filename="$(find rover_description)/urdf/rover.urdf.xacro" />
-  <xacro:include filename="$(find formulapi_gazebo)/urdf/rover.gazebo.xacro" />
+  <xacro:include filename="$(find rover_gazebo)/urdf/rover.gazebo.xacro" />
   <!-- Gazebo plugin for ROS Control -->
   <gazebo>

Commit message: initial 2d nav in gazebo

File: rover_description/urdf/rover.urdf.xacro (robot description, xacro)
@@ -88,5 +88,6 @@
     <joint name="imu_joint" type="fixed">
       <!-- <origin xyz="$(optenv HUSKY_IMU_XYZ 0.19 0 0.149)" rpy="$(optenv HUSKY_IMU_RPY 0 -1.5708 3.1416)" /> -->
-      <origin xyz="0.19 0 0.149" rpy="0 -1.5708 3.1416" />
+      <origin xyz="0.19 0 0.149" rpy="0 0 0" />
+      <!-- <origin xyz="0.19 0 0.149" rpy="0 -1.5708 3.1416" /> -->
       <parent link="base_link" />
       <child link="imu_link" />
@@ -99,5 +100,6 @@
       <parent link="base_link" />
       <child link="navsat_link" />
-      <origin xyz="0.19 0 0.149" rpy="0 -1.5708 3.1416" />
+      <origin xyz="0.19 0 0.149" rpy="0 0 0" />
+      <!-- <origin xyz="0.19 0 0.149" rpy="0 -1.5708 3.1416" /> -->
     </joint>
     <gazebo reference="navsat_link">
@@ -117,4 +119,5 @@
     </xacro:rover_wheel>
    <xacro:rover_decorate />
+    <!-- Mount a Kinect Sensor -->
     <xacro:if value="$(arg kinect_enabled)">
       <xacro:sensor_arch prefix="" parent="top_plate_link">
@@ -123,5 +126,5 @@
       <joint name="kinect_frame_joint" type="fixed">
         <!-- <origin xyz="$(optenv HUSKY_KINECT_XYZ 0 0 0)" rpy="$(optenv HUSKY_KINECT_RPY 0 0.18 3.14)" /> -->
-	<origin xyz="0 0 0" rpy="0 0.18 3.14" />
+  <origin xyz="0 0 0" rpy="0 0.18 3.14" />
         <parent link="sensor_arch_mount_link"/>
         <child link="camera_link"/>

File: rover_gazebo/urdf/rover.gazebo.xacro (robot description, xacro)
@@ -53,4 +53,17 @@
       </plugin>
     </gazebo>
+    <!-- Doesn't publish TF, just GT pose -->
+    <gazebo>
+    <plugin name="p3d_base_controller" filename="libgazebo_ros_p3d.so">
+      <alwaysOn>true</alwaysOn>
+      <updateRate>50.0</updateRate>
+      <bodyName>base_link</bodyName>
+      <topicName>ground_truth/odometry</topicName>
+      <gaussianNoise>0.01</gaussianNoise>
+      <frameName>world</frameName>
+      <xyzOffsets>0 0 0</xyzOffsets>
+      <rpyOffsets>0 0 0</rpyOffsets>
+    </plugin>
+    </gazebo>
     <xacro:if value="$(arg ur5_enabled)">
       <!--Remove when https://github.com/ros-industrial/universal_robot/pull/168 is resolved -->
