Commit message: added slam support for rc car

File: rover_description/urdf/racecar.xacro (robot description, xacro)
@@ -156,5 +156,5 @@
   <gazebo reference="imu_link">
   </gazebo>
-    <!-- Add a GPS link
+    <!-- Add a GPS link -->
     <link name="navsat_link"/>
     <joint name="navsat_joint" type="fixed">
@@ -165,5 +165,4 @@
     <gazebo reference="navsat_link">
     </gazebo>
-  -->
   <!--Mount a basic camera -->
     <xacro:camera_macro
@@ -192,6 +191,7 @@
       hz="10"
       samples="220"
+      min_range="0.1"
       >
-      <origin xyz="0.15 0 0.25" rpy="0 0 0" />
+      <origin xyz="0.2 0 0.3" rpy="0 0 0" />
     </xacro:OS1-64>
   <!-- Add Hokuyo laser scanner

Commit message: admin updates

File: rover_description/urdf/racecar.xacro (robot description, xacro)
@@ -147,13 +147,4 @@
   </joint>
   <xacro:wheel_transmission name="right_front_wheel" />
-  <!-- Add IMU link -->
-  <link name="imu_link"/>
-  <joint name="imu_joint" type="fixed">
-    <origin xyz="0.19 0 0.149" rpy="0 0 0" />
-    <parent link="chassis" />
-    <child link="imu_link" />
-  </joint>
-  <gazebo reference="imu_link">
-  </gazebo>
     <!-- Add a GPS link -->
     <link name="navsat_link"/>
@@ -187,6 +178,5 @@
     <xacro:OS1-64
       parent="chassis"
-      name="ouster"
-      topic="/os1_cloud_node/points"
+      name="os1_sensor"
       hz="10"
       samples="220"
