Commit message: added cartographer mapping supprt

File: rover_2dnav/cartographer_ros/urdf/cart_2d.urdf (robot description, URDF)
Before this commit: robot cartographer_backpack_2d, 3 links, 2 joints
Links:
- removed link os1
- added link os1_lidar; visual cylinder length=0.07 radius=0.05
Joints:
- joint os1_link_joint: child os1 -> os1_lidar
