Commit message: modifications for rc slam with teb

File: rover_2dnav/cartographer_ros/urdf/os1_sensor.urdf (robot description, URDF)
Before this commit: robot os1_sensor, 4 links, 3 joints
Links:
- removed link os1_imu
- removed link os1_lidar
Joints:
- removed joint imu_link_joint
- removed joint os1_link_joint

Commit message: minor .rviz update

File: rover_2dnav/cartographer_ros/urdf/os1_sensor.urdf (robot description, URDF)
Before this commit: robot os1_sensor, 2 links, 1 joints
Links:
- added link os1_imu; visual box size=0.06 0.04 0.02
- added link os1_lidar; visual cylinder length=0.07 radius=0.05
Joints:
- added joint imu_link_joint: type fixed, parent os1_sensor, child os1_imu, origin xyz=0.006253 -0.011775 0.007645 rpy=0 0 0
- added joint os1_link_joint: type fixed, parent os1_sensor, child os1_lidar, origin xyz=0.0 0.0 0.03618 rpy=0 0 3.14159
